File: pcb/vario.kicad_pcb (KiCad board)
At the start: 4 copper layers, 100 x 98 mm, 177 parts, among them J10 Conn_01x06, J11 Conn_01x04, J12 Conn_01x04, J13 Conn_01x04, J14 Conn_01x03, J15 Conn_01x04, J16 Conn_01x06, J17 Conn_01x06, J18 Conn_01x04, J19 Conn_01x04, J2 Conn_01x02, J20 Conn_01x06, J21 Conn_Coaxial, J22 USB_B_Micro, J23 USB_B_Micro, J24 Micro_SD_Card_Det_Hirose_DM3AT, J3 6339167-3, J6 Conn_01x06, J7 Conn_01x04, J8 Conn_01x04, J9 Conn_01x02, Q1 AO3401A, SW1 SW_MEC_5E, U1 STM32F407VGTx, U10 AMS1117-3.3, U11 HSCMRRN001PD2A3, U12 MS5611-01BA, U13 MAX3232ECPWR, U14 BLE_HM-11, U15 USBLC6-2SC6, U16 USBLC6-2SC6, U17 AMS1117-3.3, U18 HAMMOND_1593W, U2 MP2359DJ-LF-Z, U3 MP2359DJ-LF-Z, U4 L3GD20, U5 MTi-1IMU, U6 FXOS8700, U7 MS5611-01BA, U8 NEO-M9N, U9 TCAN332DR, Y1 16MHz

Commit message: started enclosure study for next version
Parts:
- removed C22, C23, C25, C27, C30, C38, C47: 100n, Capacitor_SMD:C_0402_1005Metric
- removed C24: 10n, Capacitor_SMD:C_0402_1005Metric
- removed C28, C51: 10u, Capacitor_SMD:C_1206_3216Metric
- removed C33: 4.7u, Capacitor_SMD:C_0805_2012Metric
- removed C37: 100n, Capacitor_SMD:C_0603_1608Metric
- removed D10: RED, LED_SMD:LED_0603_1608Metric
- removed J21: Conn_Coaxial, Connector_Coaxial:SMA_Molex_73251-2120_EdgeMount_Horizontal
- removed J22, J23: USB_B_Micro, Connector_USB:USB_Micro-B_Molex-105017-0001
- removed JP2: External_RF, Jumper:SolderJumper-2_P1.3mm_Bridged_Pad1.0x1.5mm
- removed L4: 27n, Inductor_SMD:L_0603_1608Metric
- removed R24: 10k, Resistor_SMD:R_0402_1005Metric
- removed R35: 1k, Resistor_SMD:R_0603_1608Metric
- removed R36: 100k, Resistor_SMD:R_0603_1608Metric
- removed R38: 10R, Resistor_SMD:R_1206_3216Metric
- removed R39, R40: 0R, Resistor_SMD:R_0603_1608Metric
- removed R41, R42: 27R, Resistor_SMD:R_0603_1608Metric
- removed TP10: GPS_SAFEBOOT, TestPoint:TestPoint_Pad_1.5x1.5mm
- removed TP11: GPS_RESETN, TestPoint:TestPoint_Pad_1.5x1.5mm
- removed TP12: GPS_LNA_EN, TestPoint:TestPoint_Pad_1.5x1.5mm
- removed U10: AMS1117-3.3, Package_TO_SOT_SMD:SOT-223-3_TabPin2
- removed U12: MS5611-01BA, Package_LGA:LGA-8_3x5mm_P1.25mm
- removed U14: BLE_HM-11, OWN_Parts_:BLE_HM-11
- removed U15: USBLC6-2SC6, Package_TO_SOT_SMD:SOT-23-6
- removed U8: NEO-M9N, RF_GPS:ublox_NEO
- added J1: RJ45-CAN, Connector_RJ:RJ45_Amphenol_RJHSE5380, F.Cu at (142.5, 149.5)
- added J4: USB_C_Receptacle_USB2.0, Connector_USB:USB_C_Receptacle_HRO_TYPE-C-31-M-12, F.Cu at (35.2, 182.6)
- J3: value 6339167-3 -> RJ45-RS232; footprint 63391673 -> Connector_RJ:RJ45_Amphenol_RJHSE5380
- R14: value 1k -> 5.11k
- R20: value 10k -> 5.11k
- R22: value 1k -> 1M
- U4: value L3GD20 -> HAMMOND_1455CF1201; footprint Package_LGA:LGA-16_4x4mm_P0.65mm_LayoutBorder4x4y -> OWN_Parts_:HAMMOND_1455CF1201
- U6: value FXOS8700 -> ESP32-WROOM-32U; footprint Package_LGA:LGA-16_3x3mm_P0.5mm_LayoutBorder3x5y -> RF_Module:ESP32-WROOM-32U
- moved R20 176.4 mm to (45.2, 184.2), turned to -90 degrees
- moved R14 172.1 mm to (47.8, 184.2), turned to -90 degrees
- moved R22 171.9 mm to (51.8, 184.0)
- moved J24 135.1 mm to (40.0, 152.6)
- moved D8 132.8 mm to (32.6, 162.9)
- moved R30 132.8 mm to (35.6, 162.9)
- moved D9 131.0 mm to (32.5, 166.3)
- moved R34 131.0 mm to (35.6, 166.3)
- moved U4 130.7 mm to (90.8, 166.5), turned to 90 degrees
- moved R37 129.6 mm to (35.7, 170.4)
- moved D11 129.6 mm to (32.6, 170.4)
- moved U1 126.3 mm to (70.1, 175.2)
- moved U5 124.1 mm to (101.0, 180.8)
- moved C50 120.9 mm to (80.9, 138.5), turned to -90 degrees
- moved U11 113.0 mm to (99.3, 156.6), turned to 180 degrees
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Connections:
- C52 pad 1: GND -> unconnected-(C52-Pad1)
- C52 pad 2: +3V3 -> unconnected-(C52-Pad2)
- R14 pad 1: Net-(R14-Pad1) -> GND
- R14 pad 2: GND -> Net-(J4-PadA5)
- R20 pad 2: FXOS8700_RST -> Net-(J4-PadB5)
- R22 pad 1: Net-(R22-Pad1) -> Net-(J4-PadS1)
- U1 pad 1: Net-(U1-Pad1) -> unconnected-(U1-Pad1)
- U1 pad 2: Net-(U1-Pad2) -> unconnected-(U1-Pad2)
- U1 pad 3: Net-(U1-Pad3) -> unconnected-(U1-Pad3)
- U1 pad 38: Net-(U1-Pad38) -> unconnected-(U1-Pad38)
- U1 pad 39: Net-(U1-Pad39) -> unconnected-(U1-Pad39)
- U1 pad 4: Net-(U1-Pad4) -> unconnected-(U1-Pad4)
- U1 pad 40: Net-(U1-Pad40) -> unconnected-(U1-Pad40)
- U1 pad 41: Net-(U1-Pad41) -> unconnected-(U1-Pad41)
- U1 pad 42: Net-(U1-Pad42) -> unconnected-(U1-Pad42)
- U1 pad 43: Net-(U1-Pad43) -> unconnected-(U1-Pad43)
- U1 pad 44: Net-(U1-Pad44) -> unconnected-(U1-Pad44)
- U1 pad 45: Net-(U1-Pad45) -> unconnected-(U1-Pad45)
- U1 pad 46: Net-(U1-Pad46) -> unconnected-(U1-Pad46)
- U1 pad 5: Net-(U1-Pad5) -> unconnected-(U1-Pad5)
- U1 pad 61: Net-(U1-Pad61) -> unconnected-(U1-Pad61)
- U1 pad 8: Net-(U1-Pad8) -> unconnected-(U1-Pad8)
- U1 pad 87: Net-(U1-Pad87) -> unconnected-(U1-Pad87)
- U1 pad 9: Net-(U1-Pad9) -> unconnected-(U1-Pad9)
- U1 pad 96: Net-(U1-Pad96) -> unconnected-(U1-Pad96)
- U1 pad 97: Net-(U1-Pad97) -> unconnected-(U1-Pad97)
- U1 pad 98: Net-(U1-Pad98) -> unconnected-(U1-Pad98)
- U11 pad 5: Net-(U11-Pad5) -> unconnected-(U11-Pad5)
- U11 pad 6: Net-(U11-Pad6) -> unconnected-(U11-Pad6)
- U11 pad 7: Net-(U11-Pad7) -> unconnected-(U11-Pad7)
- U11 pad 8: Net-(U11-Pad8) -> unconnected-(U11-Pad8)
- U5 pad 1: Net-(U5-Pad1) -> unconnected-(U5-Pad1)
- U5 pad 16: Net-(U5-Pad16) -> unconnected-(U5-Pad16)
- U5 pad 17: Net-(U5-Pad17) -> unconnected-(U5-Pad17)
- U5 pad 18: Net-(U5-Pad18) -> unconnected-(U5-Pad18)
- U5 pad 19: Net-(U5-Pad19) -> unconnected-(U5-Pad19)
- U5 pad 2: Net-(U5-Pad2) -> unconnected-(U5-Pad2)
- U5 pad 20: Net-(U5-Pad20) -> unconnected-(U5-Pad20)
- U5 pad 21: Net-(U5-Pad21) -> unconnected-(U5-Pad21)
- U5 pad 3: Net-(U5-Pad3) -> unconnected-(U5-Pad3)
- U6 pad 1: +3V3 -> Net-(U6-Pad1)
- U6 pad 10: Net-(R22-Pad1) -> unconnected-(U6-Pad10)
- U6 pad 11: FXOS8700_INT1 -> unconnected-(U6-Pad11)
- U6 pad 12: Net-(C30-Pad2) -> unconnected-(U6-Pad12)
- U6 pad 13: Net-(C30-Pad2) -> unconnected-(U6-Pad13)
- U6 pad 14: +3.3VA -> unconnected-(U6-Pad14)
- U6 pad 15: Net-(U6-Pad15) -> Net-(U6-Pad1)
- U6 pad 16: FXOS8700_RST -> unconnected-(U6-Pad16)
- U6 pad 2: Net-(C23-Pad2) -> unconnected-(U6-Pad2)
- U6 pad 3: GND -> unconnected-(U6-Pad3)
- U6 pad 4: I2C1_SCL -> unconnected-(U6-Pad4)
- U6 pad 5: GND -> unconnected-(U6-Pad5)
- U6 pad 6: I2C1_SDA -> unconnected-(U6-Pad6)
- U6 pad 7: Net-(R14-Pad1) -> unconnected-(U6-Pad7)
- U6 pad 8: Net-(C25-Pad2) -> unconnected-(U6-Pad8)
- U6 pad 9: FXOS8700_INT2 -> unconnected-(U6-Pad9)
- U7 pad 6: Net-(U7-Pad6) -> unconnected-(U7-Pad6)
- U9 pad 5: Net-(U9-Pad5) -> unconnected-(U9-Pad5)
- U9 pad 8: Net-(U9-Pad8) -> unconnected-(U9-Pad8)
Routing:
- net (no net): track 0.00 -> 232.4 mm, vias 0 -> 4
- net SPI2_MISO: track 59.7 -> 165.5 mm, vias 4 -> 12
- net L3GD20_INT2: track 55.3 -> 0.00 mm, vias 4 -> 0
- net L3GD20_INT1: track 50.6 -> 0.00 mm, vias 4 -> 0
- net USB_GPS_D+: track 44.2 -> 0.00 mm
- net USB_GPS_D-: track 43.5 -> 0.00 mm
- net Net-(C51-Pad1): track 38.5 -> 0.00 mm, vias 2 -> 0
- net Net-(JP2-Pad1): track 27.1 -> 0.00 mm, vias 2 -> 0
- net Net-(D10-Pad2): track 23.8 -> 0.00 mm
- net GND: track 330.9 -> 316.6 mm, vias 105 -> 101
- net Net-(J23-Pad6): track 14.0 -> 0.00 mm
- net Net-(J22-Pad6): track 14.0 -> 0.00 mm
- net VBUS_USB_GPS: track 110.3 -> 97.7 mm
- net Net-(R24-Pad1): track 12.3 -> 0.00 mm
- net Net-(J21-Pad1): track 12.0 -> 0.00 mm
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- added copper zone on F.Cu, net (none)
- removed copper zone on F.Cu, net Net-(C51-Pad1)
Other:
- board text added: "Pressure Connection here!"
- board text added: "SMA connectors where?"
- board text removed: "1"
- board text removed: "2"
- board text removed: "Differential Pressure"
- board text removed: "Pitot"
- board text removed: "Pressure Absolute"
