File: pcb/vario.kicad_sch (KiCad schematic)
At the start: 177 parts, among them J10 Conn_01x06, J11 Conn_01x04, J12 Conn_01x04, J13 Conn_01x04, J14 Conn_01x03, J15 Conn_01x04, J16 Conn_01x06, J17 Conn_01x06, J18 Conn_01x04, J19 Conn_01x04, J2 Conn_01x02, J20 Conn_01x06, J21 Conn_Coaxial, J22 USB_B_Micro, J23 USB_B_Micro, J24 Micro_SD_Card_Det_Hirose_DM3AT, J3 6339167-3, J6 Conn_01x06, J7 Conn_01x04, J8 Conn_01x04, J9 Conn_01x02, Q1 AO3401A, SW1 SW_MEC_5E, U1 STM32F407VGTx, U10 AMS1117-3.3, U11 HSCMRRN001PD2A3, U12 MS5611-01BA, U13 MAX3232ECPWR, U14 BLE_HM-11, U15 USBLC6-2SC6, U16 USBLC6-2SC6, U17 AMS1117-3.3, U18 HAMMOND_1593W, U2 MP2359DJ-LF-Z, U3 MP2359DJ-LF-Z, U4 L3GD20, U5 MTi-1IMU, U6 FXOS8700, U7 MS5611-01BA, U8 NEO-M9N, U9 TCAN332DR, Y1 16MHz

Commit message: started enclosure study for next version
Parts:
- removed C22, C23, C25, C27, C30, C38, C47: 100n, Capacitor_SMD:C_0402_1005Metric, symbol Device:C_Small
- removed C24: 10n, Capacitor_SMD:C_0402_1005Metric, symbol Device:C_Small
- removed C28, C51: 10u, Capacitor_SMD:C_1206_3216Metric, symbol Device:C_Small
- removed C33: 4.7u, Capacitor_SMD:C_0805_2012Metric, symbol Device:C_Small
- removed C37: 100n, Capacitor_SMD:C_0603_1608Metric, symbol Device:C_Small
- removed D10: RED, LED_SMD:LED_0603_1608Metric, symbol Device:LED_Small
- removed J21: Conn_Coaxial, Connector_Coaxial:SMA_Molex_73251-2120_EdgeMount_Horizontal, symbol Connector:Conn_Coaxial
- removed J22, J23: USB_B_Micro, Connector_USB:USB_Micro-B_Molex-105017-0001, symbol Connector:USB_B_Micro
- removed J3: 6339167-3, 63391673, symbol SamacSys_Parts:6339167-3
- removed JP2: External_RF, Jumper:SolderJumper-2_P1.3mm_Bridged_Pad1.0x1.5mm, symbol Jumper:SolderJumper_2_Bridged
- removed L4: 27n, Inductor_SMD:L_0603_1608Metric, symbol Device:L_Small
- removed R14, R22, R35: 1k, Resistor_SMD:R_0603_1608Metric, symbol Device:R_Small
- removed R20: 10k, Resistor_SMD:R_0603_1608Metric, symbol Device:R_Small
- removed R24: 10k, Resistor_SMD:R_0402_1005Metric, symbol Device:R_Small
- removed R36: 100k, Resistor_SMD:R_0603_1608Metric, symbol Device:R_Small
- removed R38: 10R, Resistor_SMD:R_1206_3216Metric, symbol Device:R_Small
- removed R39, R40: 0R, Resistor_SMD:R_0603_1608Metric, symbol Device:R_Small
- removed R41, R42: 27R, Resistor_SMD:R_0603_1608Metric, symbol Device:R_Small
- removed TP10: GPS_SAFEBOOT, TestPoint:TestPoint_Pad_1.5x1.5mm, symbol Connector:TestPoint
- removed TP11: GPS_RESETN, TestPoint:TestPoint_Pad_1.5x1.5mm, symbol Connector:TestPoint
- removed TP12: GPS_LNA_EN, TestPoint:TestPoint_Pad_1.5x1.5mm, symbol Connector:TestPoint
- removed U10: AMS1117-3.3, Package_TO_SOT_SMD:SOT-223-3_TabPin2, symbol Regulator_Linear:AMS1117-3.3
- removed U12: MS5611-01BA, Package_LGA:LGA-8_3x5mm_P1.25mm, symbol Sensor_Pressure:MS5611-01BA
- removed U14: BLE_HM-11, OWN_Parts_:BLE_HM-11, symbol OWN_Parts_:BLE_HM-11
- removed U15: USBLC6-2SC6, Package_TO_SOT_SMD:SOT-23-6, symbol Power_Protection:USBLC6-2SC6
- removed U4: L3GD20, Package_LGA:LGA-16_4x4mm_P0.65mm_LayoutBorder4x4y, symbol Sensor_Motion:L3GD20
- removed U6: FXOS8700, Package_LGA:LGA-16_3x3mm_P0.5mm_LayoutBorder3x5y, symbol OWN_Parts_:FXOS8700
- removed U8: NEO-M9N, RF_GPS:ublox_NEO, symbol RF_GPS:NEO-M8N
- added J1: RJ45-CAN, RJ45_Amphenol_RJHSE5380, symbol Connector:RJ45
- added J3: RJ45-RS232, RJ45_Amphenol_RJHSE5380, symbol Connector:RJ45
- added J?: USB_C_Receptacle_USB2.0, Connector_USB:USB_C_Receptacle_HRO_TYPE-C-31-M-12, symbol Connector:USB_C_Receptacle_USB2.0
- added R? (x2): 5.11k, Resistor_SMD:R_0603_1608Metric, symbol Device:R_Small
- added R?: 1M, Resistor_SMD:R_0603_1608Metric, symbol Device:R_Small
- added U4: HAMMOND_1455CF1201, OWN_Parts_:HAMMOND_1455CF1201, symbol OWN_Parts_:HAMMOND_1455CF1201
- added U6: ESP32-WROOM-32U, RF_Module:ESP32-WROOM-32U, symbol RF_Module:ESP32-WROOM-32U
Connections:
- net +12V: now also J1.7, J1.8, J3.7, J3.8
- net +3V3: no longer C52.2
- net CAN1H: now also J1.3
- net CAN1L: now also J1.4
- net GND: now also J1.1, J1.2, J3.1, J3.2, J?.A1 (GND), J?.A12 (GND), J?.B1 (GND), J?.B12 (GND), R?.1, R?.1, R?.2; no longer C52.1
- net RS232_1_RX: now also J3.3
- net RS232_1_TX: now also J3.4
- net USB_CONN_D+: now also J?.A6 (D+), J?.B6 (D+)
- net USB_CONN_D-: now also J?.A7 (D-), J?.B7 (D-)
- net VBUS_USB_STM32F4: now also J?.A4 (VBUS), J?.A9 (VBUS), J?.B4 (VBUS), J?.B9 (VBUS)
- new net: U6.1 (GND), U6.15 (GND), U6.38 (GND), U6.39 (GND)
- new net: J?.A5 (CC1), R?.2
- new net: J?.B5 (CC2), R?.2
- new net: J?.S1 (SHIELD), R?.1
- no-connect marks 48 -> 37
Other:
- note added: "Bluetooth / Wifi"
- note added: "Cheap IMU?"
- note added: "Main RJ45 connector"
- note removed: "Bluetooth"
- note removed: "Cheap GYRO"
- note removed: "Cheap MAG + ACC"
- note removed: "I2C Addr: 0x1E"
- note removed: "I2C Addr: 0xEC"
- note removed: "Main 4x RJ45 connector"
- note removed: "Pitot total pressure backup"
- note removed: "USB-GPS"
- moved on the sheet: C52, TP17
